Commit message: Trajectory

File: Assets/ur3e.urdf (robot description, URDF)
Before this commit: robot ur3e_robot, 11 links, 10 joints
Links:
- added link feutre_link; collision mesh filename=package://ur_description/meshes/ur3e/collision/feutre.stl; visual mesh filename=package://ur_description/meshes/ur3e/visual/feutre.dae
Joints:
- added joint tool0-feutre: type fixed, parent tool0, child feutre_link, origin xyz=0 0 0.166 rpy=0 0 0

Commit message: Menus + Trajectoire à l'envers

File: Assets/ur3e.urdf (robot description, URDF)
Before this commit: robot ur3e_robot, 12 links, 11 joints
Links:
- removed link feutre_link
Joints:
- removed joint tool0-feutre
